File: pcb/n64_gamecat_pcb/_autosave-n64_gamecat.kicad_pcb (KiCad board)
At the start: 2 copper layers, 117.5 x 162.5 mm, 12 parts

Commit message: Add rev 3 PCB
Parts:
- removed the REF** at (276.9, 68.6)
- moved REF** 6.35 mm to (144.8, 143.5)
- moved REF** 6.35 mm to (134.6, 143.5)
- moved REF** 6.35 mm to (114.3, 143.5)
- moved REF** 6.35 mm to (124.5, 143.5)
- moved REF** 6.35 mm to (114.3, 147.3)
- moved REF** 6.35 mm to (124.5, 147.3)
Routing:
- net (no net): track 6328.6 -> 6430.2 mm
