File: n64_gamecat_rp2350b/n64_gamecat_rp2350b.kicad_pcb (KiCad board)
At the start: 2 copper layers, 65 x 97 mm, 18 parts, among them J4 Conn_01x02_Pin, SW1 SW_SPDT, U3 SN74CBTLV3245ADW, U4 SN74CBTLV3245ADW

Commit message: Somewhat working with debug logging
Parts:
- removed SW1: SW_SPDT, Connector_PinSocket_2.54mm:PinSocket_1x03_P2.54mm_Vertical
- removed U3, U4: SN74CBTLV3245ADW, footprints:DW20
- added U5: SN74CB3Q3245PWR, footprints:PW20, F.Cu at (142.5, 68.5)
- added U6: SN74CB3Q3245PWR, footprints:PW20, F.Cu at (172.5, 68.5)
- moved C1 8.28 mm to (146.3, 116.9)
- moved J4 6.02 mm to (156.0, 73.7)
- moved C3 4.73 mm to (168.0, 65.5)
- moved C2 4.61 mm to (138.0, 65.5)
- moved A1 3.21 mm to (155.5, 94.0)
- moved C4 3.21 mm to (139.8, 80.4)
- moved C5 3.21 mm to (135.3, 80.9)
- moved R1 3.21 mm to (166.8, 80.4)
- moved R2 3.21 mm to (142.3, 80.4)
- moved R3 3.21 mm to (148.8, 112.9)
- moved R4 3.21 mm to (144.3, 112.9)
Routing:
- net AD4: track 126.9 -> 76.2 mm, vias 4 -> 1
- net ALE_H: track 129.8 -> 174.6 mm, vias 2 -> 5
- net AD0: track 117.6 -> 76.8 mm
- net GND: track 426.8 -> 463.6 mm, vias 7 -> 5
- net CA_AD1: track 59.7 -> 23.9 mm, vias 2 -> 0
- net AD10: track 113.8 -> 78.1 mm
- net AD11: track 115.0 -> 79.7 mm, vias 3 -> 1
- net CA_AD3: track 55.0 -> 22.2 mm, vias 1 -> 0
- net CA_AD0: track 56.9 -> 24.6 mm, vias 1 -> 0
- net CA_AD12: track 14.5 -> 45.3 mm, vias 0 -> 1
- net VSYS: track 35.3 -> 4.60 mm
- net CA_AD2: track 53.3 -> 23.1 mm, vias 1 -> 0
- net CA_AD15: track 24.9 -> 55.1 mm
- net AD7: track 107.9 -> 78.8 mm, vias 6 -> 1
- net AD3: track 98.8 -> 70.6 mm, vias 4 -> 1
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Other:
- board text added: "N64 GameCat Andrew {dblquote}CyanBlob{dblquote} Thomas 07/20/26"
- board text removed: "USB <-> N64 POWER"
