File: n64_gamecat_rp2350b/n64_gamecat_rp2350b.kicad_sch (KiCad schematic)
At the start: 18 parts, among them J4 Conn_01x02_Pin, SW1 SW_SPDT, U3 SN74CBTLV3245ADW, U4 SN74CBTLV3245ADW

Commit message: Somewhat working with debug logging
Parts:
- removed SW1: SW_SPDT, Connector_PinSocket_2.54mm:PinSocket_1x03_P2.54mm_Vertical, symbol Switch:SW_SPDT
- removed U3, U4: SN74CBTLV3245ADW, footprints:DW20, symbol 2026-04-17_18-55-28:SN74CBTLV3245ADW
- added U5, U6: SN74CB3Q3245PWR, PW20, symbol 2026-07-21_00-02-04:SN74CB3Q3245PWR
Connections:
- net 3V3_OUT: now also U5.20 (VCC), U6.20 (VCC)
- net AD0: now also U5.2 (A1)
- net AD1: now also U5.3 (A2)
- net AD10: now also U6.4 (A3)
- net AD11: now also U6.5 (A4)
- net AD12: now also U6.6 (A5)
- net AD13: now also U6.7 (A6)
- net AD14: now also U6.8 (A7)
- net AD15: now also U6.9 (A8)
- net AD2: now also U5.4 (A3)
- net AD3: now also U5.5 (A4)
- net AD4: now also U5.6 (A5)
- net AD5: now also U5.7 (A6)
- net AD6: now also U5.8 (A7)
- net AD7: now also U5.9 (A8)
- net AD8: now also U6.2 (A1)
- net AD9: now also U6.3 (A2)
- net CART_EN: now also U5.19 (*OE), U6.19 (*OE)
- net CA_AD0: now also U5.18 (B1)
- net CA_AD1: now also U5.17 (B2)
- net CA_AD10: now also U6.16 (B3)
- net CA_AD11: now also U6.15 (B4)
- net CA_AD12: now also U6.14 (B5)
- net CA_AD13: now also U6.13 (B6)
- net CA_AD14: now also U6.12 (B7)
- net CA_AD15: now also U6.11 (B8)
- net CA_AD2: now also U5.16 (B3)
- net CA_AD3: now also U5.15 (B4)
- net CA_AD4: now also U5.14 (B5)
- net CA_AD5: now also U5.13 (B6)
- net CA_AD6: now also U5.12 (B7)
- net CA_AD7: now also U5.11 (B8)
- net CA_AD8: now also U6.18 (B1)
- net CA_AD9: now also U6.17 (B2)
- net GND: now also U5.10 (GND), U6.10 (GND)
- net NC: now also U5.1 (NC), U6.1 (NC)
- no-connect marks 1 -> 0
